File: KeychainFlashLightAdvanced/KeychainFlashLightAdvanced.kicad_pcb (KiCad board)
At the start: 2 copper layers, 76.2 x 35.3 mm, 6 parts

Commit message: cleanup
Routing:
- net Net-(BT1-+): track 69.3 -> 68.1 mm
- net (no net): track 61.8 -> 61.0 mm
Changed lines of the file:
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@@
     (effects (font (size 1 1) (thickness 0.15)) (justify left bottom))
   )
-  (segment (start 75.184 67.056) (end 87.884 67.056) (width 0.25) (layer "F.Cu") (net 0))
-  (segment (start 98.044 77.216) (end 118.364 77.216) (width 0.25) (layer "F.Cu") (net 0))
-  (segment (start 87.884 67.056) (end 98.044 77.216) (width 0.25) (layer "F.Cu") (net 0))
-  (segment (start 118.364 77.216) (end 128.524 67.056) (width 0.25) (layer "F.Cu") (net 0))
-  (segment (start 128.524 54.256) (end 113.384 54.256) (width 0.25) (layer "F.Cu") (net 1))
-  (segment (start 106.1 66.5734) (end 106.1 61.54) (width 0.25) (layer "F.Cu") (net 1))
-  (segment (start 138.684 72.496) (end 138.684 61.616) (width 0.25) (layer "F.Cu") (net 1))
-  (segment (start 138.684 61.616) (end 131.424 54.356) (width 0.25) (layer "F.Cu") (net 1))
-  (segment (start 106.1 61.54) (end 113.384 54.256) (width 0.25) (layer "F.Cu") (net 1))
-  (segment (start 131.324 79.856) (end 138.684 72.496) (width 0.25) (layer "F.Cu") (net 1))
-  (segment (start 128.524 79.856) (end 131.324 79.856) (width 0.25) (layer "F.Cu") (net 1))
-  (segment (start 101.6 66.5734) (end 106.1 66.5734) (width 0.25) (layer "F.Cu") (net 1))
-  (segment (start 90.424 74.676) (end 80.264 74.676) (width 0.25) (layer "F.Cu") (net 3))
-  (segment (start 80.264 74.676) (end 75.184 69.596) (width 0.25) (layer "F.Cu") (net 3))
-  (segment (start 93.0426 64.516) (end 101.6 73.0734) (width 0.25) (layer "F.Cu") (net 5))
-  (segment (start 106.1 73.0734) (end 101.6 73.0734) (width 0.25) (layer "F.Cu") (net 5))
-  (segment (start 90.424 64.516) (end 93.0426 64.516) (width 0.25) (layer "F.Cu") (net 5))
+  (segment (start 85.630036 67.056) (end 75.184 67.056) (width 0.25) (layer "F.Cu") (net 0))
+  (segment (start 100.297963 77.216) (end 116.110036 77.216) (width 0.25) (layer "F.Cu") (net 0))
+  (segment (start 96.450207 75.622207) (end 89.477792 68.649792) (width 0.25) (layer "F.Cu") (net 0))
+  (segment (start 119.957792 75.622207) (end 128.524 67.056) (width 0.25) (layer "F.Cu") (net 0))
+  (arc (start 96.450207 75.622207) (mid 98.215572 76.801786) (end 100.297963 77.216) (width 0.25) (layer "F.Cu") (net 0))
+  (arc (start 119.957792 75.622207) (mid 118.192426 76.801786) (end 116.110036 77.216) (width 0.25) (layer "F.Cu") (net 0))
+  (arc (start 89.477792 68.649792) (mid 87.712426 67.470213) (end 85.630036 67.056) (width 0.25) (layer "F.Cu") (net 0))
+  (segment (start 115.637963 54.256) (end 128.524 54.256) (width 0.25) (layer "F.Cu") (net 1))
+  (segment (start 106.1 66.5734) (end 106.1 63.793963) (width 0.25) (layer "F.Cu") (net 1))
+  (segment (start 138.684 63.869963) (end 138.684 70.242036) (width 0.25) (layer "F.Cu") (net 1))
+  (segment (start 137.090207 60.022207) (end 131.424 54.356) (width 0.25) (layer "F.Cu") (net 1))
+  (segment (start 111.790207 55.849792) (end 107.693792 59.946207) (width 0.25) (layer "F.Cu") (net 1))
+  (segment (start 132.313949 78.86605) (end 137.090207 74.089792) (width 0.25) (layer "F.Cu") (net 1))
+  (segment (start 129.924 79.856) (end 128.524 79.856) (width 0.25) (layer "F.Cu") (net 1))
+  (segment (start 106.1 66.5734) (end 101.6 66.5734) (width 0.25) (layer "F.Cu") (net 1))
+  (arc (start 132.313949 78.86605) (mid 131.217431 79.59872) (end 129.924 79.856) (width 0.25) (layer "F.Cu") (net 1))
+  (arc (start 138.684 70.242036) (mid 138.269786 72.324426) (end 137.090207 74.089792) (width 0.25) (layer "F.Cu") (net 1))
+  (arc (start 107.693792 59.946207) (mid 106.514213 61.711572) (end 106.1 63.793963) (width 0.25) (layer "F.Cu") (net 1))
+  (arc (start 137.090207 60.022207) (mid 138.269786 61.787572) (end 138.684 63.869963) (width 0.25) (layer "F.Cu") (net 1))
+  (arc (start 115.637963 54.256) (mid 113.555572 54.670213) (end 111.790207 55.849792) (width 0.25) (layer "F.Cu") (net 1))
+  (segment (start 82.517963 74.676) (end 90.424 74.676) (width 0.25) (layer "F.Cu") (net 3))
+  (segment (start 78.670207 73.082207) (end 75.184 69.596) (width 0.25) (layer "F.Cu") (net 3))
+  (arc (start 78.670207 73.082207) (mid 80.435572 74.261786) (end 82.517963 74.676) (width 0.25) (layer "F.Cu") (net 3))
+  (segment (start 101.6 73.0734) (end 93.968414 65.441814) (width 0.25) (layer "F.Cu") (net 5))
+  (segment (start 101.6 73.0734) (end 106.1 73.0734) (width 0.25) (layer "F.Cu") (net 5))
+  (segment (start 91.7333 64.516) (end 90.424 64.516) (width 0.25) (layer "F.Cu") (net 5))
+  (arc (start 93.968414 65.441814) (mid 92.942935 64.756611) (end 91.7333 64.516) (width 0.25) (layer "F.Cu") (net 5))
 )
