File: KeychainFlashLightIntroduction/KeychainFlashLightIntroduction.kicad_sch (KiCad schematic)
At the start: 4 parts, among them SW1 SW_DPST_x2

Commit message: Added "blanc" workshop files and cheatsheets
Parts:
- removed BT1: Battery_Cell, Battery:BatteryHolder_Keystone_3002_1x2032, symbol Device:Battery_Cell
- removed D1: LED, LED_THT:LED_D5.0mm_Clear, symbol Device:LED
- removed R1: R, Resistor_THT:R_Axial_DIN0207_L6.3mm_D2.5mm_P10.16mm_Horizontal, symbol Device:R
- removed SW1: SW_DPST_x2, Button_Switch_THT:SW_Tactile_Straight_KSA0Axx1LFTR, symbol Switch:SW_DPST_x2
Changed lines of the file:
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@@
 (kicad_sch (version 20230121) (generator eeschema)
   (paper "A4")
-  (wire (pts (xy 148.59 91.44) (xy 154.94 91.44))
-    (stroke (width 0) (type default))
-  )
-  (wire (pts (xy 120.65 91.44) (xy 120.65 105.41))
-    (stroke (width 0) (type default))
-  )
-  (wire (pts (xy 133.35 105.41) (xy 139.7 105.41))
-    (stroke (width 0) (type default))
-  )
-  (wire (pts (xy 154.94 105.41) (xy 149.86 105.41))
-    (stroke (width 0) (type default))
-  )
-  (wire (pts (xy 125.73 91.44) (xy 120.65 91.44))
-    (stroke (width 0) (type default))
-  )
-  (wire (pts (xy 154.94 91.44) (xy 154.94 105.41))
-    (stroke (width 0) (type default))
-  )
-  (wire (pts (xy 133.35 91.44) (xy 140.97 91.44))
-    (stroke (width 0) (type default))
-  )
-  (wire (pts (xy 120.65 105.41) (xy 125.73 105.41))
-    (stroke (width 0) (type default))
-  )
-  (symbol (lib_id "Switch:SW_DPST_x2") (at 144.78 105.41 0) (unit 1)
-    (in_bom yes) (on_board yes) (dnp no) (fields_autoplaced)
-    (property "Reference" "SW1" (at 144.78 99.06 0)
-      (effects (font (size 1.27 1.27)))
-    )
-    (property "Value" "SW_DPST_x2" (at 144.78 101.6 0)
-      (effects (font (size 1.27 1.27)))
-    )
-    (property "Footprint" "Button_Switch_THT:SW_Tactile_Straight_KSA0Axx1LFTR" (at 144.78 105.41 0)
-      (effects (font (size 1.27 1.27)) hide)
-    )
-    (property "Datasheet" "~" (at 144.78 105.41 0)
-      (effects (font (size 1.27 1.27)) hide)
-    )
-    (pin "1")
-    (pin "2")
-    (pin "3")
-    (pin "4")
-    (instances
-      (project "KeychainFlashLight"
-        (path "/30398b8a-8fed-4ca8-b3cc-b1f61d914000"
-          (reference "SW1") (unit 1)
-        )
-      )
-    )
-  )
-  (symbol (lib_id "Device:R") (at 144.78 91.44 90) (unit 1)
-    (in_bom yes) (on_board yes) (dnp no) (fields_autoplaced)
-    (property "Reference" "R1" (at 144.78 85.09 90)
-      (effects (font (size 1.27 1.27)))
-    )
-    (property "Value" "R" (at 144.78 87.63 90)
-      (effects (font (size 1.27 1.27)))
-    )
-    (property "Footprint" "Resistor_THT:R_Axial_DIN0207_L6.3mm_D2.5mm_P10.16mm_Horizontal" (at 144.78 93.218 90)
-      (effects (font (size 1.27 1.27)) hide)
-    )
-    (property "Datasheet" "~" (at 144.78 91.44 0)
-      (effects (font (size 1.27 1.27)) hide)
-    )
-    (pin "1")
-    (pin "2")
-    (instances
-      (project "KeychainFlashLight"
-        (path "/30398b8a-8fed-4ca8-b3cc-b1f61d914000"
-          (reference "R1") (unit 1)
-        )
-      )
-    )
-  )
-  (symbol (lib_id "Device:LED") (at 129.54 91.44 0) (unit 1)
-    (in_bom yes) (on_board yes) (dnp no) (fields_autoplaced)
-    (property "Reference" "D1" (at 127.9525 85.09 0)
-      (effects (font (size 1.27 1.27)))
-    )
-    (property "Value" "LED" (at 127.9525 87.63 0)
-      (effects (font (size 1.27 1.27)))
-    )
-    (property "Footprint" "LED_THT:LED_D5.0mm_Clear" (at 129.54 91.44 0)
-      (effects (font (size 1.27 1.27)) hide)
-    )
-    (property "Datasheet" "~" (at 129.54 91.44 0)
-      (effects (font (size 1.27 1.27)) hide)
-    )
-    (pin "1")
-    (pin "2")
-    (instances
-      (project "KeychainFlashLight"
-        (path "/30398b8a-8fed-4ca8-b3cc-b1f61d914000"
-          (reference "D1") (unit 1)
-        )
-      )
-    )
-  )
-  (symbol (lib_id "Device:Battery_Cell") (at 128.27 105.41 270) (unit 1)
-    (in_bom yes) (on_board yes) (dnp no) (fields_autoplaced)
-    (property "Reference" "BT1" (at 130.1115 97.79 90)
-      (effects (font (size 1.27 1.27)))
-    )
-    (property "Value" "Battery_Cell" (at 130.1115 100.33 90)
-      (effects (font (size 1.27 1.27)))
-    )
-    (property "Footprint" "Battery:BatteryHolder_Keystone_3002_1x2032" (at 129.794 105.41 90)
-      (effects (font (size 1.27 1.27)) hide)
-    )
-    (property "Datasheet" "~" (at 129.794 105.41 90)
-      (effects (font (size 1.27 1.27)) hide)
-    )
-    (pin "1")
-    (pin "2")
-    (instances
-      (project "KeychainFlashLight"
-        (path "/30398b8a-8fed-4ca8-b3cc-b1f61d914000"
-          (reference "BT1") (unit 1)
-        )
-      )
-    )
-  )
   (sheet_instances
     (path "/" (page "1"))
