File: Finished Workshops (review form or cheatsheet)/KeychainFlashLightAdvanced (Finished)/KeychainFlashLightAdvanced.kicad_pcb (KiCad board)
At the start: 2 copper layers, 76.2 x 35.3 mm, 6 parts

Commit message: Updated Advanced workshop, cleanup
Both workshops now been updated with latest feedback
Parts:
- moved REF** 2.29 mm to (129.5, 73.0)
Connections:
- BT1 pad 2: +3.3V -> GND
Routing:
- net GND: track 0.00 -> 61.0 mm
- net (no net): track 61.0 -> 0.00 mm
Changed lines of the file:
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@@
   (net 0 "")
   (net 1 "Net-(BT1-+)")
-  (net 2 "+3.3V")
-  (net 3 "Net-(D1-A)")
-  (net 4 "GND")
-  (net 5 "Net-(R1-Pad2)")
+  (net 2 "Net-(D1-A)")
+  (net 3 "GND")
+  (net 4 "Net-(R1-Pad2)")
   (footprint "Battery:BatteryHolder_Keystone_3002_1x2032" (layer "F.Cu")
     (at 128.524 67.056 -90)
@@
       (net 1 "Net-(BT1-+)") (pinfunction "+") (pintype "passive"))
     (pad "2" smd circle (at 0 0 270) (size 17.8 17.8) (layers "F.Cu" "F.Mask")
-      (net 2 "+3.3V") (pinfunction "-") (pintype "passive"))
+      (net 3 "GND") (pinfunction "-") (pintype "passive"))
     (model "${KICAD7_3DMODEL_DIR}/Battery.3dshapes/BatteryHolder_Keystone_3034_1x20mm.step"
       (offset (xyz 0 0 0))
@@
       (net 1 "Net-(BT1-+)") (pintype "passive") (solder_mask_margin 0.102))
     (pad "3" thru_hole circle (at 3.25 -2.25 270) (size 1.498 1.498) (drill 0.99) (layers "*.Cu" "*.Mask")
-      (net 5 "Net-(R1-Pad2)") (pintype "passive") (solder_mask_margin 0.102))
+      (net 4 "Net-(R1-Pad2)") (pintype "passive") (solder_mask_margin 0.102))
     (pad "4" thru_hole circle (at 3.25 2.25 270) (size 1.498 1.498) (drill 0.99) (layers "*.Cu" "*.Mask")
-      (net 5 "Net-(R1-Pad2)") (pintype "passive") (solder_mask_margin 0.102))
+      (net 4 "Net-(R1-Pad2)") (pintype "passive") (solder_mask_margin 0.102))
     (model "${KIPRJMOD}/3D-models/FSM8JH--3DModel-STEP-56544.STEP"
       (offset (xyz 0 0 0))
@@
       (stroke (width 0.1) (type solid)) (layer "F.Fab"))
     (pad "1" thru_hole circle (at 0 0 90) (size 1.6 1.6) (drill 0.8) (layers "*.Cu" "*.Mask")
-      (net 3 "Net-(D1-A)") (pintype "passive"))
+      (net 2 "Net-(D1-A)") (pintype "passive"))
     (pad "2" thru_hole oval (at 10.16 0 90) (size 1.6 1.6) (drill 0.8) (layers "*.Cu" "*.Mask")
-      (net 5 "Net-(R1-Pad2)") (pintype "passive"))
+      (net 4 "Net-(R1-Pad2)") (pintype "passive"))
     (model "${KICAD6_3DMODEL_DIR}/Resistor_THT.3dshapes/R_Axial_DIN0207_L6.3mm_D2.5mm_P10.16mm_Horizontal.wrl"
       (offset (xyz 0 0 0))
@@
       (stroke (width 0.1) (type solid)) (fill none) (layer "F.Fab"))
     (pad "1" thru_hole rect (at 0 0 270) (size 1.8 1.8) (drill 0.9) (layers "*.Cu" "*.Mask")
-      (net 4 "GND") (pinfunction "K") (pintype "passive"))
+      (net 3 "GND") (pinfunction "K") (pintype "passive"))
     (pad "2" thru_hole circle (at 2.54 0 270) (size 1.8 1.8) (drill 0.9) (layers "*.Cu" "*.Mask")
-      (net 3 "Net-(D1-A)") (pinfunction "A") (pintype "passive"))
+      (net 2 "Net-(D1-A)") (pinfunction "A") (pintype "passive"))
     (model "${KICAD6_3DMODEL_DIR}/LED_THT.3dshapes/LED_D5.0mm_Clear.wrl"
       (offset (xyz 0 0 -3))
@@
   )
   (footprint "Symbol:OSHW-Logo2_24.3x20mm_SilkScreen" (layer "B.Cu")
-    (at 128.27 71.12 180)
+    (at 129.54 73.025 180)
     (descr "Open Source Hardware Symbol")
     (tags "Logo Symbol OSHW")
@@
     (effects (font (size 1 1) (thickness 0.15)) (justify left bottom))
   )
-  (segment (start 85.630036 67.056) (end 75.184 67.056) (width 0.25) (layer "F.Cu") (net 0))
-  (segment (start 100.297963 77.216) (end 116.110036 77.216) (width 0.25) (layer "F.Cu") (net 0))
-  (segment (start 96.450207 75.622207) (end 89.477792 68.649792) (width 0.25) (layer "F.Cu") (net 0))
-  (segment (start 119.957792 75.622207) (end 128.524 67.056) (width 0.25) (layer "F.Cu") (net 0))
-  (arc (start 96.450207 75.622207) (mid 98.215572 76.801786) (end 100.297963 77.216) (width 0.25) (layer "F.Cu") (net 0))
-  (arc (start 119.957792 75.622207) (mid 118.192426 76.801786) (end 116.110036 77.216) (width 0.25) (layer "F.Cu") (net 0))
-  (arc (start 89.477792 68.649792) (mid 87.712426 67.470213) (end 85.630036 67.056) (width 0.25) (layer "F.Cu") (net 0))
   (segment (start 115.637963 54.256) (end 128.524 54.256) (width 0.25) (layer "F.Cu") (net 1))
   (segment (start 106.1 66.5734) (end 106.1 63.793963) (width 0.25) (layer "F.Cu") (net 1))
@@
   (arc (start 137.090207 60.022207) (mid 138.269786 61.787572) (end 138.684 63.869963) (width 0.25) (layer "F.Cu") (net 1))
   (arc (start 115.637963 54.256) (mid 113.555572 54.670213) (end 111.790207 55.849792) (width 0.25) (layer "F.Cu") (net 1))
-  (segment (start 82.517963 74.676) (end 90.424 74.676) (width 0.25) (layer "F.Cu") (net 3))
-  (segment (start 78.670207 73.082207) (end 75.184 69.596) (width 0.25) (layer "F.Cu") (net 3))
-  (arc (start 78.670207 73.082207) (mid 80.435572 74.261786) (end 82.517963 74.676) (width 0.25) (layer "F.Cu") (net 3))
-  (segment (start 101.6 73.0734) (end 93.968414 65.441814) (width 0.25) (layer "F.Cu") (net 5))
-  (segment (start 101.6 73.0734) (end 106.1 73.0734) (width 0.25) (layer "F.Cu") (net 5))
-  (segment (start 91.7333 64.516) (end 90.424 64.516) (width 0.25) (layer "F.Cu") (net 5))
-  (arc (start 93.968414 65.441814) (mid 92.942935 64.756611) (end 91.7333 64.516) (width 0.25) (layer "F.Cu") (net 5))
+  (segment (start 82.517963 74.676) (end 90.424 74.676) (width 0.25) (layer "F.Cu") (net 2))
+  (segment (start 78.670207 73.082207) (end 75.184 69.596) (width 0.25) (layer "F.Cu") (net 2))
+  (arc (start 78.670207 73.082207) (mid 80.435572 74.261786) (end 82.517963 74.676) (width 0.25) (layer "F.Cu") (net 2))
+  (segment (start 85.630036 67.056) (end 75.184 67.056) (width 0.25) (layer "F.Cu") (net 3))
+  (segment (start 100.297963 77.216) (end 116.110036 77.216) (width 0.25) (layer "F.Cu") (net 3))
+  (segment (start 96.450207 75.622207) (end 89.477792 68.649792) (width 0.25) (layer "F.Cu") (net 3))
+  (segment (start 119.957792 75.622207) (end 128.524 67.056) (width 0.25) (layer "F.Cu") (net 3))
+  (arc (start 96.450207 75.622207) (mid 98.215572 76.801786) (end 100.297963 77.216) (width 0.25) (layer "F.Cu") (net 3))
+  (arc (start 119.957792 75.622207) (mid 118.192426 76.801786) (end 116.110036 77.216) (width 0.25) (layer "F.Cu") (net 3))
+  (arc (start 89.477792 68.649792) (mid 87.712426 67.470213) (end 85.630036 67.056) (width 0.25) (layer "F.Cu") (net 3))
+  (segment (start 101.6 73.0734) (end 93.968414 65.441814) (width 0.25) (layer "F.Cu") (net 4))
+  (segment (start 101.6 73.0734) (end 106.1 73.0734) (width 0.25) (layer "F.Cu") (net 4))
+  (segment (start 91.7333 64.516) (end 90.424 64.516) (width 0.25) (layer "F.Cu") (net 4))
+  (arc (start 93.968414 65.441814) (mid 92.942935 64.756611) (end 91.7333 64.516) (width 0.25) (layer "F.Cu") (net 4))
 )
