File: Finished Workshops (review form or cheatsheet)/KeychainFlashLightAdvanced (Finished)/flashlightmodule.kicad_sch (KiCad schematic)
At the start: 4 parts

Commit message: Updated Advanced workshop, cleanup
Both workshops now been updated with latest feedback
Connections:
- net GND is gone; now on net 3.3V Input: D1.1 (K)
Changed lines of the file:
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@@
     (comment 1 "Made By: Casper Tak")
+  )
+  (junction (at 140.97 106.68) (diameter 0) (color 0 0 0 0)
   )
   (junction (at 156.21 106.68) (diameter 0) (color 0 0 0 0)
   )
+  (junction (at 140.97 92.71) (diameter 0) (color 0 0 0 0)
+  )
   (junction (at 168.91 106.68) (diameter 0) (color 0 0 0 0)
+  )
+  (wire (pts (xy 140.97 106.68) (xy 142.24 106.68))
+    (stroke (width 0) (type default))
+  )
+  (wire (pts (xy 140.97 92.71) (xy 140.97 106.68))
+    (stroke (width 0) (type default))
   )
   (wire (pts (xy 149.86 106.68) (xy 156.21 106.68))
@@
     (stroke (width 0) (type default))
   )
+  (wire (pts (xy 139.7 106.68) (xy 140.97 106.68))
+    (stroke (width 0) (type default))
+  )
   (wire (pts (xy 171.45 106.68) (xy 168.91 106.68))
+    (stroke (width 0) (type default))
+  )
+  (wire (pts (xy 139.7 92.71) (xy 140.97 92.71))
+    (stroke (width 0) (type default))
+  )
+  (wire (pts (xy 140.97 92.71) (xy 142.24 92.71))
     (stroke (width 0) (type default))
   )
@@
     (effects (font (size 1.27 1.27)) (justify left bottom))
   )
-  (hierarchical_label "3.3V Input" (shape input) (at 142.24 106.68 180) (fields_autoplaced)
+  (hierarchical_label "3.3V Input" (shape input) (at 139.7 106.68 180) (fields_autoplaced)
     (effects (font (size 1.27 1.27)) (justify right))
   )
-  (hierarchical_label "GND" (shape input) (at 142.24 92.71 180) (fields_autoplaced)
+  (hierarchical_label "GND" (shape input) (at 139.7 92.71 180) (fields_autoplaced)
     (effects (font (size 1.27 1.27)) (justify right))
   )
